File: pcbs/mackerel/mackerel.kicad_pcb (KiCad board)
At the start: 2 copper layers, 129.5 x 97.8 mm, 60 parts, among them J1 MJ-4PP-9-kbd-corne-light-resc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, SW1 SW_Push, SW10 SW_Push, SW11 SW_Push, SW12 SW_Push, SW13 SW_Push, SW14 SW_Push, SW15 SW_Push, SW16 SW_Push, SW17 SW_Push, SW18 SW_Push, SW19 SW_Push, SW2 SW_Push, SW20 SW_Push, SW21 SW_Push, SW22 SW_Push, SW23 SW_Push, SW24 SW_Push, SW25 SW_Push, SW26 SW_Push, SW27 SW_Push, SW28 SW_Push, SW29 SW_Push, SW3 SW_Push, SW4 SW_Push, SW5 SW_Push, SW6 SW_Push, SW7 SW_Push, SW8 SW_Push, SW9 SW_Push, U1 rp2040-zero

Commit message: updates
Parts:
- added REF**: MountingHole_2.7mm_M2.5_ISO7380, MountingHole:MountingHole_2.7mm_M2.5_ISO7380, F.Cu at (117.0, 39.6)
- added REF**: MountingHole_2.7mm_M2.5_ISO7380, MountingHole:MountingHole_2.7mm_M2.5_ISO7380, F.Cu at (27.4, 76.5)
- added REF**: MountingHole_2.7mm_M2.5_ISO7380, MountingHole:MountingHole_2.7mm_M2.5_ISO7380, F.Cu at (127.6, 113.4)
Routing:
- net /ROW4: track 160.7 -> 161.4 mm

Commit message: licenses
Connections:
- J1 pad B: /RX -> /TX
Routing:
- net /TX: track 0.00 -> 106.2 mm, vias 0 -> 4
- net /RX: track 101.6 -> 0.00 mm, vias 3 -> 0
- net /COL4: track 245.5 -> 243.6 mm
- net GND: track 102.9 -> 101.8 mm, vias 4 -> 3
- net /COL1: track 186.0 -> 184.9 mm
- net /COL5: track 206.3 -> 207.2 mm
- net /ROW4: track 161.4 -> 162.3 mm
