File: pcbs/mackerel/mackerel.kicad_sch (KiCad schematic)
At the start: 60 parts, among them J1 MJ-4PP-9-kbd-corne-light-resc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, SW1 SW_Push, SW10 SW_Push, SW11 SW_Push, SW12 SW_Push, SW13 SW_Push, SW14 SW_Push, SW15 SW_Push, SW16 SW_Push, SW17 SW_Push, SW18 SW_Push, SW19 SW_Push, SW2 SW_Push, SW20 SW_Push, SW21 SW_Push, SW22 SW_Push, SW23 SW_Push, SW24 SW_Push, SW25 SW_Push, SW26 SW_Push, SW27 SW_Push, SW28 SW_Push, SW29 SW_Push, SW3 SW_Push, SW4 SW_Push, SW5 SW_Push, SW6 SW_Push, SW7 SW_Push, SW8 SW_Push, SW9 SW_Push, U1 rp2040-zero

Commit message: Update
Parts:
- U1: footprint mackerel:rp2040-zero-smd_modified-semi-reversible -> mackerel:rp2040-zero-tht_modified-semi-reversible
Changed lines of the file:
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@@
 			)
 		)
-		(property "Footprint" "mackerel:rp2040-zero-smd_modified-semi-reversible"
+		(property "Footprint" "mackerel:rp2040-zero-tht_modified-semi-reversible"
 			(at 182.88 59.69 0)
 			(effects

Commit message: licenses
Parts:
- added H1, H2, H3: MountingHole, symbol Mechanical:MountingHole
Connections:
- net TX: now reaches U1.1 (0)
- net TX: now also J1.B
- net RX: no longer names the net of U1.2 (1)
- net RX: no longer J1.B
Changed lines of the file:
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@@
 	)
 	(no_connect
-		(at 204.47 55.88)
+		(at 204.47 58.42)
 	)
 	(wire
@@
 	(wire
 		(pts
+			(xy 204.47 55.88) (xy 210.82 55.88)
+		)
+		(stroke
+			(width 0)
+			(type default)
+		)
+	)
+	(wire
+		(pts
 			(xy 121.92 48.26) (xy 121.92 63.5)
 		)
@@
 	(wire
 		(pts
-			(xy 204.47 58.42) (xy 210.82 58.42)
-		)
-		(stroke
-			(width 0)
-			(type default)
-		)
-	)
-	(wire
-		(pts
 			(xy 86.36 101.6) (xy 101.6 101.6)
 		)
@@
 		)
 	)
-	(label "RX"
-		(at 210.82 58.42 0)
+	(label "TX"
+		(at 210.82 55.88 0)
 		(fields_autoplaced yes)
 		(effects
@@
 		)
 	)
-	(label "RX"
+	(label "TX"
 		(at 198.12 115.57 0)
 		(fields_autoplaced yes)
@@
 	)
 	(symbol
+		(lib_id "Mechanical:MountingHole")
+		(at 153.67 50.8 0)
+		(unit 1)
+		(exclude_from_sim yes)
+		(in_bom no)
+		(on_board yes)
+		(dnp no)
+		(fields_autoplaced yes)
+		(property "Reference" "H3"
+			(at 156.21 49.5299 0)
+			(effects
+				(font
+					(size 1.27 1.27)
+				)
+				(justify left)
+			)
+		)
+		(property "Value" "MountingHole"
+			(at 156.21 52.0699 0)
+			(effects
+				(font
+					(size 1.27 1.27)
+				)
+				(justify left)
+			)
+		)
+		(property "Footprint" ""
+			(at 153.67 50.8 0)
+			(effects
+				(font
+					(size 1.27 1.27)
+				)
+				(hide yes)
+			)
+		)
+		(property "Datasheet" "~"
+			(at 153.67 50.8 0)
+			(effects
+				(font
+					(size 1.27 1.27)
+				)
+				(hide yes)
+			)
+		)
+		(property "Description" "Mounting Hole without connection"
+			(at 153.67 50.8 0)
+			(effects
+				(font
+					(size 1.27 1.27)
+				)
+				(hide yes)
+			)
+		)
+		(instances
+			(project "mackerel"
+				(path "/1717b0a7-21a3-4878-a536-f4352e8f0c36"
+					(reference "H3")
+					(unit 1)
+				)
+			)
+		)
+	)
+	(symbol
 		(lib_id "Switch:SW_Push")
 		(at 50.8 78.74 0)
@@
 	)
 	(symbol
+		(lib_id "Mechanical:MountingHole")
+		(at 153.67 45.72 0)
+		(unit 1)
+		(exclude_from_sim yes)
+		(in_bom no)
+		(on_board yes)
+		(dnp no)
+		(fields_autoplaced yes)
+		(property "Reference" "H2"
+			(at 156.21 44.4499 0)
+			(effects
+				(font
+					(size 1.27 1.27)
+				)
+				(justify left)
+			)
+		)
+		(property "Value" "MountingHole"
+			(at 156.21 46.9899 0)
+			(effects
+				(font
+					(size 1.27 1.27)
+				)
+				(justify left)
+			)
+		)
+		(property "Footprint" ""
+			(at 153.67 45.72 0)
+			(effects
+				(font
+					(size 1.27 1.27)
+				)
+				(hide yes)
+			)
+		)
+		(property "Datasheet" "~"
+			(at 153.67 45.72 0)
+			(effects
+				(font
+					(size 1.27 1.27)
+				)
+				(hide yes)
+			)
+		)
+		(property "Description" "Mounting Hole without connection"
+			(at 153.67 45.72 0)
+			(effects
+				(font
+					(size 1.27 1.27)
+				)
+				(hide yes)
+			)
+		)
+		(instances
+			(project "mackerel"
+				(path "/1717b0a7-21a3-4878-a536-f4352e8f0c36"
+					(reference "H2")
+					(unit 1)
+				)
+			)
+		)
+	)
+	(symbol
 		(lib_id "Switch:SW_Push")
 		(at 96.52 93.98 0)
@@
 					(unit 1)
 				)
+			)
+		)
+	)
+	(symbol
+		(lib_id "Mechanical:MountingHole")
+		(at 153.67 40.64 0)
+		(unit 1)
+		(exclude_from_sim yes)
+		(in_bom no)
+		(on_board yes)
+		(dnp no)
+		(fields_autoplaced yes)
+		(property "Reference" "H1"
+			(at 156.21 39.3699 0)
+			(effects
+				(font
+					(size 1.27 1.27)
+				)
+				(justify left)
+			)
+		)
+		(property "Value" "MountingHole"
+			(at 156.21 41.9099 0)
+			(effects
+				(font
+					(size 1.27 1.27)
+				)
+				(justify left)
+			)
+		)
+		(property "Footprint" ""
+			(at 153.67 40.64 0)
+			(effects
+				(font
+					(size 1.27 1.27)
+				)
+				(hide yes)
+			)
+		)
+		(property "Datasheet" "~"
+			(at 153.67 40.64 0)
+			(effects
+				(font
+					(size 1.27 1.27)
+				)
+				(hide yes)
+			)
+		)
+		(property "Description" "Mounting Hole without connection"
+			(at 153.67 40.64 0)
+			(effects
+				(font
+					(size 1.27 1.27)
+				)
+				(hide yes)
+			)
+		)
+		(instances
+			(project ""
+				(path "/1717b0a7-21a3-4878-a536-f4352e8f0c36"
+					(reference "H1")
+					(unit 1)
+				)
